Commit message: add all 4 wheels to holonomic urdf

File: urdf/holo.urdf.xacro (robot description, xacro)
@@ -11,4 +11,6 @@
   <xacro:property name="base_side_length" value="0.5" />
   <xacro:property name="wheel_offset" value="${ (((base_side_length * base_side_length)/2) ** 0.5)/2}" />
+  <xacro:property name="wheel_width" value = "${0.05}"/>
+  <xacro:property name="wheel_width_offset" value = "${ (((wheel_width/2) * (wheel_width/2))/2) ** 0.5}"/>
   <link name="base_link">
     <visual>
@@ -26,8 +28,44 @@
     <visual>
       <geometry>
-        <cylinder radius = "0.1" length = "0.05"/>
+        <cylinder radius = "0.075" length = "0.05"/>
       </geometry>
       <material name = "black"/>
-      <origin xyz = "${wheel_offset} ${wheel_offset} 0.05" rpy = "0 ${pi/2} ${pi/4}"/>
+      <origin xyz = "${wheel_offset + wheel_width_offset} ${wheel_offset + wheel_width_offset} -0.075" rpy = "0 ${pi/2} ${pi/4}"/>
+    </visual>
+    <collision>
+      <box size = "0.5 0.5 0.2"/>
+    </collision>
+  </link>
+  <link name="right_back_wheel">
+    <visual>
+      <geometry>
+        <cylinder radius = "0.075" length = "0.05"/>
+      </geometry>
+      <material name = "black"/>
+      <origin xyz = "${wheel_offset + wheel_width_offset} ${-wheel_offset - wheel_width_offset} -0.075" rpy = "0 ${pi/2} ${pi/4}"/>
+    </visual>
+    <collision>
+      <box size = "0.5 0.5 0.2"/>
+    </collision>
+  </link>
+  <link name="left_front_wheel">
+    <visual>
+      <geometry>
+        <cylinder radius = "0.075" length = "0.05"/>
+      </geometry>
+      <material name = "black"/>
+      <origin xyz = "${-wheel_offset - wheel_width_offset} ${wheel_offset + wheel_width_offset} -0.075" rpy = "0 ${pi/2} ${pi/4}"/>
+    </visual>
+    <collision>
+      <box size = "0.5 0.5 0.2"/>
+    </collision>
+  </link>
+  <link name="left_back_wheel">
+    <visual>
+      <geometry>
+        <cylinder radius = "0.075" length = "0.05"/>
+      </geometry>
+      <material name = "black"/>
+      <origin xyz = "${- wheel_offset - wheel_width_offset} ${-wheel_offset - wheel_width_offset} -0.075" rpy = "0 ${pi/2} ${pi/4}"/>
     </visual>
     <collision>

Commit message: try to get wheel transmission/joint working

File: urdf/holo.urdf.xacro (robot description, xacro)
@@ -22,5 +22,7 @@
     </visual>
     <collision>
-      <box size = "0.5 0.5 0.2"/>
+      <geometry>
+        <box size = "${base_side_length} ${base_side_length} 0.2"/>
+      </geometry>
     </collision>
   </link>
@@ -34,8 +36,26 @@
     </visual>
     <collision>
-      <box size = "0.5 0.5 0.2"/>
+     <geometry>
+        <cylinder radius = "0.075" length = "0.05"/>
+      </geometry>
+      <origin xyz = "${wheel_offset + wheel_width_offset} ${wheel_offset + wheel_width_offset} -0.075" rpy = "0 ${pi/2} ${pi/4}"/>
     </collision>
   </link>
-  <link name="right_back_wheel">
+  <joint name="right_front_wheel_joint" type="continuous">
+    <parent link="base_link"/>
+    <child link="right_front_wheel"/>
+    <origin xyz = "${wheel_offset + wheel_width_offset} ${wheel_offset + wheel_width_offset} -0.075" rpy = "0 ${pi/2} ${pi/4}"/>
+    <axis xyz ="${wheel_offset + wheel_width_offset} ${wheel_offset + wheel_width_offset} 0"/>
+  </joint>
+  <transmission name="right_front_wheel_trans">
+    <type>transmission_interface/SimpleTransmission</type>
+    <actuator name="right_front_wheel_motor">
+      <mechanicalReduction>1</mechanicalReduction>
+    </actuator>
+    <joint name="right_front_wheel_joint">
+      <hardwareInterface>hardware_interface/VelocityJointInterface</hardwareInterface>
+    </joint>
+  </transmission>
+  <!-- <link name="right_back_wheel">
     <visual>
       <geometry>
@@ -72,4 +92,9 @@
       <box size = "0.5 0.5 0.2"/>
     </collision>
-  </link>
+  </link> -->
+  <gazebo>
+    <plugin name="gazebo_ros_control" filename="libgazebo_ros_control.so">
+      <robotNamespace>/</robotNamespace>
+    </plugin>
+  </gazebo>
 </robot>

Commit message: still complaining about a missing transform and joint

File: urdf/holo.urdf.xacro (robot description, xacro)
@@ -25,4 +25,5 @@
         <box size = "${base_side_length} ${base_side_length} 0.2"/>
       </geometry>
+      <origin rpy = "0 0 ${pi/4}"/>
     </collision>
   </link>
@@ -37,5 +38,5 @@
     <collision>
      <geometry>
-        <cylinder radius = "0.075" length = "0.05"/>
+        <cylinder radius = "0.075" length = "0.04"/>
       </geometry>
       <origin xyz = "${wheel_offset + wheel_width_offset} ${wheel_offset + wheel_width_offset} -0.075" rpy = "0 ${pi/2} ${pi/4}"/>
@@ -45,6 +46,6 @@
     <parent link="base_link"/>
     <child link="right_front_wheel"/>
-    <origin xyz = "${wheel_offset + wheel_width_offset} ${wheel_offset + wheel_width_offset} -0.075" rpy = "0 ${pi/2} ${pi/4}"/>
-    <axis xyz ="${wheel_offset + wheel_width_offset} ${wheel_offset + wheel_width_offset} 0"/>
+    <!-- <origin xyz = "${wheel_offset + wheel_width_offset} ${wheel_offset + wheel_width_offset} -0.075" rpy = "0 ${pi/2} ${pi/4}"/> -->
+    <axis xyz ="1 1 0"/>
   </joint>
   <transmission name="right_front_wheel_trans">

Commit message: remove the wheel, add a turret that should function, testing tbd

File: urdf/holo.urdf.xacro (robot description, xacro)
@@ -7,4 +7,10 @@
     <color rgba="0 0 0 1"/>
   </material>
+  <xacro:macro name="default_inertial" params="mass">
+    <inertial>
+      <mass value="${mass}" />
+      <inertia ixx="1.0" ixy="0.0" ixz="0.0" iyy="1.0" iyz="0.0" izz="1.0" />
+    </inertial>
+  </xacro:macro>
 <!-- x axis red, y axis green -->
   <xacro:property name="pi" value="3.1415926" />
@@ -27,5 +33,40 @@
       <origin rpy = "0 0 ${pi/4}"/>
     </collision>
+    <xacro:default_inertial mass="10"/>
   </link>
+  <link name="turret">
+    <visual>
+      <geometry>
+        <cylinder radius="0.25" length="0.1"/>
+      </geometry>
+      <origin xyz="0.0 0.0 0"/>
+    </visual>
+    <collision>
+      <geometry>
+        <cylinder radius="0.25" length="0.1"/>
+        <origin xyz="0.0 0.0 0.15"/>
+      </geometry>
+    </collision>
+    <xacro:default_inertial mass="2"/>
+  </link>
+  <joint name="turret_joint" type="continuous">
+    <parent link="base_link"/>
+    <child link="turret"/>
+    <origin xyz="0.0 0.0 0.15"/>
+    <axis xyz="0.0 0.0 1"/>
+    <limit effort="30" velocity="1.0"/>
+    <dynamics damping="0.0" friction="0.0"/>
+    <kp value = '1'/>
+  </joint>
+  <transmission name="turret_swivel_trans">
+    <type>transmission_interface/SimpleTransmission</type>
+    <actuator name="$turret_swivel_motor">
+      <mechanicalReduction>1</mechanicalReduction>
+    </actuator>
+    <joint name="turret_joint">
+      <hardwareInterface>VelocityJointInterface</hardwareInterface>
+    </joint>
+  </transmission>
+<!--
   <link name="right_front_wheel">
     <visual>
@@ -46,5 +87,5 @@
     <parent link="base_link"/>
     <child link="right_front_wheel"/>
-    <!-- <origin xyz = "${wheel_offset + wheel_width_offset} ${wheel_offset + wheel_width_offset} -0.075" rpy = "0 ${pi/2} ${pi/4}"/> -->
+    <origin xyz = "${wheel_offset + wheel_width_offset} ${wheel_offset + wheel_width_offset} -0.075" rpy = "0 0 9"/>
     <axis xyz ="1 1 0"/>
   </joint>
@@ -57,5 +98,5 @@
       <hardwareInterface>hardware_interface/VelocityJointInterface</hardwareInterface>
     </joint>
-  </transmission>
+  </transmission> -->
   <!-- <link name="right_back_wheel">
     <visual>

Commit message: turret spins

File: urdf/holo.urdf.xacro (robot description, xacro)
@@ -40,10 +40,8 @@
         <cylinder radius="0.25" length="0.1"/>
       </geometry>
-      <origin xyz="0.0 0.0 0"/>
     </visual>
     <collision>
       <geometry>
         <cylinder radius="0.25" length="0.1"/>
-        <origin xyz="0.0 0.0 0.15"/>
       </geometry>
     </collision>
@@ -68,4 +66,23 @@
     </joint>
   </transmission>
+  <link name="turret_bar">
+    <visual>
+      <geometry>
+        <box size="0.7 0.1 0.1"/>
+      </geometry>
+      <material name="white">
+      </material>
+    </visual>
+      <collision>
+        <geometry>
+        <box size="0.7 0.1 0.1"/>
+      </geometry>
+    </collision>
+  </link>
+  <joint name="turret_to_bar_link" type="fixed">
+    <parent link="turret"/>
+    <child link="turret_bar"/>
+    <origin xyz="0.0 0.0 0.1"/>
+  </joint>
 <!--
   <link name="right_front_wheel">

Commit message: launch file and rviz work properly now

File: urdf/holo.urdf.xacro (robot description, xacro)
@@ -25,5 +25,5 @@
       </geometry>
       <material name = "white"/>
-      <origin rpy = "0 0 ${pi/4}"/>
+      <origin xyz = "0 0 0" rpy = "0 0 ${pi/4}"/>
     </visual>
     <collision>
@@ -31,7 +31,7 @@
         <box size = "${base_side_length} ${base_side_length} 0.2"/>
       </geometry>
-      <origin rpy = "0 0 ${pi/4}"/>
+      <origin xyz = "0 0 0" rpy = "0 0 ${pi/4}"/>
     </collision>
-    <xacro:default_inertial mass="10"/>
+    <xacro:default_inertial mass="8"/>
   </link>
   <link name="turret">
@@ -71,6 +71,5 @@
         <box size="0.7 0.1 0.1"/>
       </geometry>
-      <material name="white">
-      </material>
+      <material name="white"/>
     </visual>
       <collision>

Commit message: wheel 1 works (but goes backwards)

File: urdf/holo.urdf.xacro (robot description, xacro)
@@ -55,5 +55,5 @@
     <limit effort="30" velocity="1.0"/>
     <dynamics damping="0.0" friction="0.0"/>
-    <kp value = '1'/>
+    <!-- <kp value = '1'/> -->
   </joint>
   <transmission name="turret_swivel_trans">
@@ -84,5 +84,4 @@
     <origin xyz="0.0 0.0 0.1"/>
   </joint>
-<!--
   <link name="right_front_wheel">
     <visual>
@@ -91,5 +90,6 @@
       </geometry>
       <material name = "black"/>
-      <origin xyz = "${wheel_offset + wheel_width_offset} ${wheel_offset + wheel_width_offset} -0.075" rpy = "0 ${pi/2} ${pi/4}"/>
+      <!-- <origin xyz = "${wheel_offset + wheel_width_offset} ${wheel_offset + wheel_width_offset} -0.075" rpy = "0 ${pi/2} ${pi/4}"/> -->
+      <origin rpy="0 ${pi/2} ${pi/4}"/>
     </visual>
     <collision>
@@ -97,22 +97,27 @@
         <cylinder radius = "0.075" length = "0.04"/>
       </geometry>
-      <origin xyz = "${wheel_offset + wheel_width_offset} ${wheel_offset + wheel_width_offset} -0.075" rpy = "0 ${pi/2} ${pi/4}"/>
+      <!-- <origin xyz = "${wheel_offset + wheel_width_offset} ${wheel_offset + wheel_width_offset} -0.075" rpy = "0 ${pi/2} ${pi/4}"/> -->
+      <origin rpy="0 ${pi/2} ${pi/4}"/>
     </collision>
+    <xacro:default_inertial mass="1"/>
   </link>
   <joint name="right_front_wheel_joint" type="continuous">
     <parent link="base_link"/>
     <child link="right_front_wheel"/>
-    <origin xyz = "${wheel_offset + wheel_width_offset} ${wheel_offset + wheel_width_offset} -0.075" rpy = "0 0 9"/>
+    <!-- <origin xyz = "${wheel_offset + wheel_width_offset} ${wheel_offset + wheel_width_offset} -0.075" rpy = "0 ${pi/2} ${pi/4}"/> -->
+    <origin xyz = "${wheel_offset + wheel_width_offset} ${wheel_offset + wheel_width_offset} -0.075"/>
     <axis xyz ="1 1 0"/>
+    <limit effort="60" velocity="6.0"/>
+    <dynamics damping="0.0" friction="0.0"/>
   </joint>
   <transmission name="right_front_wheel_trans">
-    <type>transmission_interface/SimpleTransmission</type>
+    <type>SimpleTransmission</type>
     <actuator name="right_front_wheel_motor">
       <mechanicalReduction>1</mechanicalReduction>
     </actuator>
     <joint name="right_front_wheel_joint">
-      <hardwareInterface>hardware_interface/VelocityJointInterface</hardwareInterface>
+      <hardwareInterface>VelocityJointInterface</hardwareInterface>
     </joint>
-  </transmission> -->
+  </transmission>
   <!-- <link name="right_back_wheel">
     <visual>

Commit message: all wheel exist, 2 of 4 confirmed to work

File: urdf/holo.urdf.xacro (robot description, xacro)
@@ -90,12 +90,10 @@
       </geometry>
       <material name = "black"/>
-      <!-- <origin xyz = "${wheel_offset + wheel_width_offset} ${wheel_offset + wheel_width_offset} -0.075" rpy = "0 ${pi/2} ${pi/4}"/> -->
-      <origin rpy="0 ${pi/2} ${pi/4}"/>
-    </visual>
-    <collision>
-     <geometry>
-        <cylinder radius = "0.075" length = "0.04"/>
-      </geometry>
-      <!-- <origin xyz = "${wheel_offset + wheel_width_offset} ${wheel_offset + wheel_width_offset} -0.075" rpy = "0 ${pi/2} ${pi/4}"/> -->
+      <origin rpy="0 ${pi/2} ${pi/4}"/>
+    </visual>
+    <collision>
+     <geometry>
+        <cylinder radius = "0.075" length = "0.04"/>
+      </geometry>
       <origin rpy="0 ${pi/2} ${pi/4}"/>
     </collision>
@@ -105,5 +103,4 @@
     <parent link="base_link"/>
     <child link="right_front_wheel"/>
-    <!-- <origin xyz = "${wheel_offset + wheel_width_offset} ${wheel_offset + wheel_width_offset} -0.075" rpy = "0 ${pi/2} ${pi/4}"/> -->
     <origin xyz = "${wheel_offset + wheel_width_offset} ${wheel_offset + wheel_width_offset} -0.075"/>
     <axis xyz ="1 1 0"/>
@@ -120,16 +117,4 @@
     </joint>
   </transmission>
-  <!-- <link name="right_back_wheel">
-    <visual>
-      <geometry>
-        <cylinder radius = "0.075" length = "0.05"/>
-      </geometry>
-      <material name = "black"/>
-      <origin xyz = "${wheel_offset + wheel_width_offset} ${-wheel_offset - wheel_width_offset} -0.075" rpy = "0 ${pi/2} ${pi/4}"/>
-    </visual>
-    <collision>
-      <box size = "0.5 0.5 0.2"/>
-    </collision>
-  </link>
   <link name="left_front_wheel">
     <visual>
@@ -138,10 +123,31 @@
       </geometry>
       <material name = "black"/>
-      <origin xyz = "${-wheel_offset - wheel_width_offset} ${wheel_offset + wheel_width_offset} -0.075" rpy = "0 ${pi/2} ${pi/4}"/>
-    </visual>
-    <collision>
-      <box size = "0.5 0.5 0.2"/>
-    </collision>
-  </link>
+      <origin rpy="0 ${pi/2} ${-pi/4}"/>
+    </visual>
+    <collision>
+     <geometry>
+        <cylinder radius = "0.075" length = "0.04"/>
+      </geometry>
+      <origin rpy="0 ${pi/2} ${-pi/4}"/>
+    </collision>
+    <xacro:default_inertial mass="1"/>
+  </link>
+  <joint name="left_front_wheel_joint" type="continuous">
+    <parent link="base_link"/>
+    <child link="left_front_wheel"/>
+    <origin xyz = "${- wheel_offset - wheel_width_offset} ${wheel_offset + wheel_width_offset} -0.075"/>
+    <axis xyz ="-1 1 0"/>
+    <limit effort="60" velocity="6.0"/>
+    <dynamics damping="0.0" friction="0.0"/>
+  </joint>
+  <transmission name="left_front_wheel_trans">
+    <type>SimpleTransmission</type>
+    <actuator name="left_front_wheel_motor">
+      <mechanicalReduction>1</mechanicalReduction>
+    </actuator>
+    <joint name="left_front_wheel_joint">
+      <hardwareInterface>VelocityJointInterface</hardwareInterface>
+    </joint>
+  </transmission>
   <link name="left_back_wheel">
     <visual>
@@ -150,10 +156,64 @@
       </geometry>
       <material name = "black"/>
-      <origin xyz = "${- wheel_offset - wheel_width_offset} ${-wheel_offset - wheel_width_offset} -0.075" rpy = "0 ${pi/2} ${pi/4}"/>
-    </visual>
-    <collision>
-      <box size = "0.5 0.5 0.2"/>
-    </collision>
-  </link> -->
+      <origin rpy="0 ${pi/2} ${pi/4}"/>
+    </visual>
+    <collision>
+     <geometry>
+        <cylinder radius = "0.075" length = "0.04"/>
+      </geometry>
+      <origin rpy="0 ${pi/2} ${pi/4}"/>
+    </collision>
+    <xacro:default_inertial mass="1"/>
+  </link>
+  <joint name="left_back_wheel_joint" type="continuous">
+    <parent link="base_link"/>
+    <child link="left_back_wheel"/>
+    <origin xyz = "${- wheel_offset - wheel_width_offset} ${-wheel_offset - wheel_width_offset} -0.075"/>
+    <axis xyz ="-1 -1 0"/>
+    <limit effort="60" velocity="6.0"/>
+    <dynamics damping="0.0" friction="0.0"/>
+  </joint>
+  <transmission name="left_back_wheel_trans">
+    <type>SimpleTransmission</type>
+    <actuator name="left_back_wheel_motor">
+      <mechanicalReduction>1</mechanicalReduction>
+    </actuator>
+    <joint name="left_back_wheel_joint">
+      <hardwareInterface>VelocityJointInterface</hardwareInterface>
+    </joint>
+  </transmission>
+  <link name="right_back_wheel">
+    <visual>
+      <geometry>
+        <cylinder radius = "0.075" length = "0.05"/>
+      </geometry>
+      <material name = "black"/>
+      <origin rpy="0 ${pi/2} ${-pi/4}"/>
+    </visual>
+    <collision>
+     <geometry>
+        <cylinder radius = "0.075" length = "0.04"/>
+      </geometry>
+      <origin rpy="0 ${pi/2} ${-pi/4}"/>
+    </collision>
+    <xacro:default_inertial mass="1"/>
+  </link>
+  <joint name="right_back_wheel_joint" type="continuous">
+    <parent link="base_link"/>
+    <child link="right_back_wheel"/>
+    <origin xyz = "${wheel_offset + wheel_width_offset} ${-wheel_offset - wheel_width_offset} -0.075"/>
+    <axis xyz ="1 -1 0"/>
+    <limit effort="60" velocity="6.0"/>
+    <dynamics damping="0.0" friction="0.0"/>
+  </joint>
+  <transmission name="right_back_wheel_trans">
+    <type>SimpleTransmission</type>
+    <actuator name="right_back_wheel_motor">
+      <mechanicalReduction>1</mechanicalReduction>
+    </actuator>
+    <joint name="right_back_wheel_joint">
+      <hardwareInterface>VelocityJointInterface</hardwareInterface>
+    </joint>
+  </transmission>
   <gazebo>
     <plugin name="gazebo_ros_control" filename="libgazebo_ros_control.so">

Commit message: robot go vroom (kinda unstable though)

File: urdf/holo.urdf.xacro (robot description, xacro)
@@ -15,5 +15,5 @@
 <!-- x axis red, y axis green -->
   <xacro:property name="pi" value="3.1415926" />
-  <xacro:property name="base_side_length" value="0.5" />
+  <xacro:property name="base_side_length" value="1" />
   <xacro:property name="wheel_offset" value="${ (((base_side_length * base_side_length)/2) ** 0.5)/2}" />
   <xacro:property name="wheel_width" value = "${0.05}"/>
@@ -72,4 +72,5 @@
       </geometry>
       <material name="white"/>
+      <origin rpy="0.0 0.0 ${pi/2}"/>
     </visual>
       <collision>
@@ -77,4 +78,5 @@
         <box size="0.7 0.1 0.1"/>
       </geometry>
+      <origin rpy="0.0 0.0 ${pi/2}"/>
     </collision>
   </link>
@@ -82,5 +84,5 @@
     <parent link="turret"/>
     <child link="turret_bar"/>
-    <origin xyz="0.0 0.0 0.1"/>
+    <origin xyz="0 0.25 0.1"/>
   </joint>
   <link name="right_front_wheel">
@@ -90,11 +92,11 @@
       </geometry>
       <material name = "black"/>
-      <origin rpy="0 ${pi/2} ${pi/4}"/>
-    </visual>
-    <collision>
-     <geometry>
-        <cylinder radius = "0.075" length = "0.04"/>
-      </geometry>
-      <origin rpy="0 ${pi/2} ${pi/4}"/>
+      <origin rpy="0 ${pi/2} ${(pi/4) + pi}"/>
+    </visual>
+    <collision>
+     <geometry>
+        <cylinder radius = "0.075" length = "0.04"/>
+      </geometry>
+      <origin rpy="0 ${pi/2} ${(pi/4) + pi}"/>
     </collision>
     <xacro:default_inertial mass="1"/>
@@ -105,6 +107,6 @@
     <origin xyz = "${wheel_offset + wheel_width_offset} ${wheel_offset + wheel_width_offset} -0.075"/>
     <axis xyz ="1 1 0"/>
-    <limit effort="60" velocity="6.0"/>
-    <dynamics damping="0.0" friction="0.0"/>
+    <limit effort="30" velocity="100"/>
+    <dynamics damping="0.0" friction="0.1"/>
   </joint>
   <transmission name="right_front_wheel_trans">
@@ -138,6 +140,6 @@
     <origin xyz = "${- wheel_offset - wheel_width_offset} ${wheel_offset + wheel_width_offset} -0.075"/>
     <axis xyz ="-1 1 0"/>
-    <limit effort="60" velocity="6.0"/>
-    <dynamics damping="0.0" friction="0.0"/>
+    <limit effort="30" velocity="100"/>
+    <dynamics damping="0.0" friction="0.1"/>
   </joint>
   <transmission name="left_front_wheel_trans">
@@ -171,6 +173,6 @@
     <origin xyz = "${- wheel_offset - wheel_width_offset} ${-wheel_offset - wheel_width_offset} -0.075"/>
     <axis xyz ="-1 -1 0"/>
-    <limit effort="60" velocity="6.0"/>
-    <dynamics damping="0.0" friction="0.0"/>
+    <limit effort="30" velocity="100"/>
+    <dynamics damping="0.0" friction="0.1"/>
   </joint>
   <transmission name="left_back_wheel_trans">
@@ -189,11 +191,11 @@
       </geometry>
       <material name = "black"/>
-      <origin rpy="0 ${pi/2} ${-pi/4}"/>
-    </visual>
-    <collision>
-     <geometry>
-        <cylinder radius = "0.075" length = "0.04"/>
-      </geometry>
-      <origin rpy="0 ${pi/2} ${-pi/4}"/>
+      <origin rpy="0 ${pi/2} ${(-pi/4) + (pi)}"/>
+    </visual>
+    <collision>
+     <geometry>
+        <cylinder radius = "0.075" length = "0.04"/>
+      </geometry>
+      <origin rpy="0 ${pi/2} ${(-pi/4) + pi}"/>
     </collision>
     <xacro:default_inertial mass="1"/>
@@ -204,6 +206,6 @@
     <origin xyz = "${wheel_offset + wheel_width_offset} ${-wheel_offset - wheel_width_offset} -0.075"/>
     <axis xyz ="1 -1 0"/>
-    <limit effort="60" velocity="6.0"/>
-    <dynamics damping="0.0" friction="0.0"/>
+    <limit effort="30" velocity="100"/>
+    <dynamics damping="0.0" friction="0.1"/>
   </joint>
   <transmission name="right_back_wheel_trans">
