Commit message: more messing with the urdf, still not driving straight, not sure how big of a problem it will be

File: urdf/holo.urdf.xacro (robot description, xacro)
@@ -14,5 +14,5 @@
   </xacro:macro>
 <!-- x axis red, y axis green -->
-  <xacro:property name="pi" value="3.1415926" />
+  <!-- <xacro:property name="pi" value="3.1415926" /> -->
   <xacro:property name="base_side_length" value="1" />
   <xacro:property name="wheel_offset" value="${ (((base_side_length * base_side_length)/2) ** 0.5)/2}" />
@@ -46,5 +46,5 @@
       </geometry>
     </collision>
-    <xacro:default_inertial mass="2"/>
+    <xacro:default_inertial mass="1"/>
   </link>
   <joint name="turret_joint" type="continuous">
@@ -54,5 +54,5 @@
     <axis xyz="0.0 0.0 1"/>
     <limit effort="30" velocity="1.0"/>
-    <dynamics damping="0.0" friction="0.0"/>
+    <dynamics damping="0.0" friction="0.1"/>
     <!-- <kp value = '1'/> -->
   </joint>
@@ -96,5 +96,5 @@
     <collision>
      <geometry>
-        <cylinder radius = "0.075" length = "0.04"/>
+        <cylinder radius = "0.075" length = "0.05"/>
       </geometry>
       <origin rpy="0 ${pi/2} ${(pi/4) + pi}"/>
@@ -108,5 +108,5 @@
     <axis xyz ="1 1 0"/>
     <limit effort="30" velocity="100"/>
-    <dynamics damping="0.0" friction="0.1"/>
+    <dynamics damping="0.0" friction="0.0"/>
   </joint>
   <transmission name="right_front_wheel_trans">
@@ -129,5 +129,5 @@
     <collision>
      <geometry>
-        <cylinder radius = "0.075" length = "0.04"/>
+        <cylinder radius = "0.075" length = "0.05"/>
       </geometry>
       <origin rpy="0 ${pi/2} ${-pi/4}"/>
@@ -141,5 +141,5 @@
     <axis xyz ="-1 1 0"/>
     <limit effort="30" velocity="100"/>
-    <dynamics damping="0.0" friction="0.1"/>
+    <dynamics damping="0.0" friction="0.0"/>
   </joint>
   <transmission name="left_front_wheel_trans">
@@ -162,5 +162,5 @@
     <collision>
      <geometry>
-        <cylinder radius = "0.075" length = "0.04"/>
+        <cylinder radius = "0.075" length = "0.05"/>
       </geometry>
       <origin rpy="0 ${pi/2} ${pi/4}"/>
@@ -174,5 +174,5 @@
     <axis xyz ="-1 -1 0"/>
     <limit effort="30" velocity="100"/>
-    <dynamics damping="0.0" friction="0.1"/>
+    <dynamics damping="0.0" friction="0.0"/>
   </joint>
   <transmission name="left_back_wheel_trans">
@@ -195,5 +195,5 @@
     <collision>
      <geometry>
-        <cylinder radius = "0.075" length = "0.04"/>
+        <cylinder radius = "0.075" length = "0.05"/>
       </geometry>
       <origin rpy="0 ${pi/2} ${(-pi/4) + pi}"/>
@@ -207,5 +207,5 @@
     <axis xyz ="1 -1 0"/>
     <limit effort="30" velocity="100"/>
-    <dynamics damping="0.0" friction="0.1"/>
+    <dynamics damping="0.0" friction="0.0"/>
   </joint>
   <transmission name="right_back_wheel_trans">
