Commit message: load bixi urdf into gazebo

File: urdf/bixi/urdf/base.urdf.xacro (robot description, xacro)
@@ -2,5 +2,5 @@
 <!-- Revolute-Revolute Manipulator -->
 <robot name="bixi" xmlns:xacro="http://www.ros.org/wiki/xacro">
-    <xacro:include filename="$(find bixi_description)/urdf/wheel.urdf.xacro" />
+    <xacro:include filename="$(find urdf_sim_tutorial)/urdf/bixi/urdf/wheel.urdf.xacro" />
     <!-- Constants for robot dimensions -->
     <xacro:property name="M_PI" value="3.1415926535897931"/>
@@ -22,5 +22,5 @@
             <origin xyz="0 0 0" rpy="0 0 0" />
             <geometry>
-                <mesh filename="package://bixi_description/meshes/chasis.dae" scale="1 1 1" />
+                <mesh filename="package://urdf_sim_tutorial/urdf/bixi/meshes/chasis.dae" scale="1 1 1" />
             </geometry>
         </visual>

File: urdf/bixi/urdf/wheel.urdf.xacro (robot description, xacro)
@@ -21,8 +21,8 @@
                 <geometry>
                     <xacro:unless value="${ccw == 0}">
-                        <mesh filename="package://bixi_description/meshes/mec_f_l.dae" scale="1 1 1"/>
+                        <mesh filename="package://urdf_sim_tutorial/urdf/bixi/meshes/mec_f_l.dae" scale="1 1 1"/>
                     </xacro:unless>
                     <xacro:if value="${ccw == 0}">
-                        <mesh filename="package://bixi_description/meshes/mec_f_r.dae" scale="1 1 1"/>
+                        <mesh filename="package://urdf_sim_tutorial/urdf/bixi/meshes/mec_f_r.dae" scale="1 1 1"/>
                     </xacro:if>
                 </geometry>
